File: keypad/matrix.kicad_sch (KiCad schematic)
At the start: 38 parts, among them SW1 num, SW10 #5, SW11 #6, SW12 plu1, SW13 #1, SW14 #2, SW15 #3, SW16 ent0, SW17 #0, SW18 kom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

Commit message: Assign Footprints
Parts:
- D1, D10, D11, D12, D13, D14, D15, D16, D17, D18, D19, D2, D3, D4, D5, D6, D7, D8, D9: footprint (none) -> Diode_SMD:D_SOD-123
- SW1, SW10, SW11, SW12, SW13, SW14, SW15, SW16, SW18, SW19, SW2, SW3, SW4, SW5, SW6, SW7, SW8, SW9: footprint (none) -> Alps_Only:ALPS-1U
- SW17: footprint (none) -> Alps_Only:ALPS-2U
