File: keypad/keypad.kicad_pcb (KiCad board)
At the start: 2 copper layers, 78.6 x 111.1 mm, 59 parts, among them J1 AVR-ISP-6, SW1 num, SW10 #5, SW11 #6, SW12 plu1, SW13 #1, SW14 #2, SW15 #3, SW16 ent0, SW17 #0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

Commit message: Routed crystal oscillator
Parts:
- moved C1 5.56 mm to (71.2, 66.0)
- moved C2 5.39 mm to (74.8, 66.0), turned to -90 degrees
- moved C6 3.37 mm to (77.9, 60.2)
Routing:
- net GND: track 0.00 -> 26.9 mm
- net /XTAL1: track 0.00 -> 13.4 mm
- net /XTAL2: track 0.00 -> 12.6 mm
- net +5V: track 0.00 -> 7.86 mm
Changed lines of the file:
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@@
   )
   (footprint "Capacitor_SMD:C_0805_2012Metric_Pad1.18x1.45mm_HandSolder" (layer "B.Cu")
-    (at 68.48125 61.214 -90)
+    (at 71.247 66.04 -90)
     (descr "Capacitor SMD 0805 (2012 Metric), square (rectangular) end terminal, IPC_7351 nominal with elongated pad for handsoldering. (Body size source: IPC-SM-782 page 76, https://www.pcb-3d.com/wordpress/wp-content/uploads/ipc-sm-782a_amendment_1_and_2.pdf, https://docs.google.com/spreadsheets/d/1BsfQQcO9C6DZCsRaXUlFlo91Tg2WpOkGARC1WS5S8t0/edit?usp=sharing), generated with kicad-footprint-generator")
     (tags "capacitor handsolder")
@@
   )
   (footprint "Capacitor_SMD:C_0805_2012Metric_Pad1.18x1.45mm_HandSolder" (layer "B.Cu")
-    (at 77.2125 61.214 90)
+    (at 74.803 66.04 -90)
     (descr "Capacitor SMD 0805 (2012 Metric), square (rectangular) end terminal, IPC_7351 nominal with elongated pad for handsoldering. (Body size source: IPC-SM-782 page 76, https://www.pcb-3d.com/wordpress/wp-content/uploads/ipc-sm-782a_amendment_1_and_2.pdf, https://docs.google.com/spreadsheets/d/1BsfQQcO9C6DZCsRaXUlFlo91Tg2WpOkGARC1WS5S8t0/edit?usp=sharing), generated with kicad-footprint-generator")
     (tags "capacitor handsolder")
@@
     (property "Sheetname" "")
     (attr smd)
-    (fp_text reference "C2" (at 3.175 0 90) (layer "B.SilkS")
-      (effects (font (size 1 1) (thickness 0.15)) (justify mirror))
-    )
-    (fp_text value "22p" (at 5.55625 0 90) (layer "B.Fab")
+    (fp_text reference "C2" (at 0 1.905 90) (layer "B.SilkS")
+      (effects (font (size 1 1) (thickness 0.15)) (justify mirror))
+    )
+    (fp_text value "22p" (at -3.556 0.127 90) (layer "B.Fab")
       (effects (font (size 1 1) (thickness 0.15)) (justify mirror))
     )
@@
     (fp_line (start -1 -0.625) (end -1 0.625) (layer "B.Fab") (width 0.1))
     (fp_line (start -1 0.625) (end 1 0.625) (layer "B.Fab") (width 0.1))
-    (pad "1" smd roundrect (at -1.0375 0 90) (size 1.175 1.45) (layers "B.Cu" "B.Paste" "B.Mask") (roundrect_rratio 0.212766)
+    (pad "1" smd roundrect (at -1.0375 0 270) (size 1.175 1.45) (layers "B.Cu" "B.Paste" "B.Mask") (roundrect_rratio 0.212766)
       (net 3 "/XTAL2") (pintype "passive"))
-    (pad "2" smd roundrect (at 1.0375 0 90) (size 1.175 1.45) (layers "B.Cu" "B.Paste" "B.Mask") (roundrect_rratio 0.212766)
+    (pad "2" smd roundrect (at 1.0375 0 270) (size 1.175 1.45) (layers "B.Cu" "B.Paste" "B.Mask") (roundrect_rratio 0.212766)
       (net 2 "GND") (pintype "passive"))
     (model "${KICAD6_3DMODEL_DIR}/Capacitor_SMD.3dshapes/C_0805_2012Metric.wrl"
@@
   )
   (footprint "Capacitor_SMD:C_0805_2012Metric_Pad1.18x1.45mm_HandSolder" (layer "B.Cu")
-    (at 77.9835 56.82675 180)
+    (at 77.851 60.198 180)
     (descr "Capacitor SMD 0805 (2012 Metric), square (rectangular) end terminal, IPC_7351 nominal with elongated pad for handsoldering. (Body size source: IPC-SM-782 page 76, https://www.pcb-3d.com/wordpress/wp-content/uploads/ipc-sm-782a_amendment_1_and_2.pdf, https://docs.google.com/spreadsheets/d/1BsfQQcO9C6DZCsRaXUlFlo91Tg2WpOkGARC1WS5S8t0/edit?usp=sharing), generated with kicad-footprint-generator")
     (tags "capacitor handsolder")
@@
   (gr_line (start 37.30625 149.225) (end 110.33125 149.225) (layer "Edge.Cuts") (width 0.1))
   (gr_line (start 114.3 53.18125) (end 112.7125 53.18125) (layer "Edge.Cuts") (width 0.1))
+  (segment (start 69.977 61.341) (end 71.04775 60.27025) (width 0.25) (layer "B.Cu") (net 1))
+  (segment (start 73.221 57.335) (end 73.221 54.033) (width 0.25) (layer "B.Cu") (net 1))
+  (segment (start 71.56625 58.98975) (end 73.221 57.335) (width 0.25) (layer "B.Cu") (net 1))
+  (segment (start 69.977 64.135) (end 69.977 61.341) (width 0.25) (layer "B.Cu") (net 1))
+  (segment (start 71.04775 60.27025) (end 71.56625 60.27025) (width 0.25) (layer "B.Cu") (net 1))
+  (segment (start 71.56625 58.98975) (end 71.56625 60.27025) (width 0.25) (layer "B.Cu") (net 1))
+  (segment (start 70.8445 65.0025) (end 69.977 64.135) (width 0.25) (layer "B.Cu") (net 1))
+  (segment (start 71.247 65.0025) (end 70.8445 65.0025) (width 0.25) (layer "B.Cu") (net 1))
+  (segment (start 74.821 57.420604) (end 75.248198 57.847802) (width 0.25) (layer "B.Cu") (net 2))
+  (segment (start 74.803 67.0775) (end 76.8135 65.067) (width 0.25) (layer "B.Cu") (net 2))
+  (segment (start 76.8135 59.413104) (end 75.248198 57.847802) (width 0.25) (layer "B.Cu") (net 2))
+  (segment (start 76.8135 60.198) (end 76.8135 59.413104) (width 0.25) (layer "B.Cu") (net 2))
+  (segment (start 74.31625 60.27025) (end 72.01625 62.57025) (width 0.25) (layer "B.Cu") (net 2))
+  (segment (start 73.025 64.029) (end 71.56625 62.57025) (width 0.25) (layer "B.Cu") (net 2))
+  (segment (start 72.01625 62.57025) (end 71.56625 62.57025) (width 0.25) (layer "B.Cu") (net 2))
+  (segment (start 74.46625 60.27025) (end 74.31625 60.27025) (width 0.25) (layer "B.Cu") (net 2))
+  (segment (start 73.025 65.2995) (end 74.803 67.0775) (width 0.25) (layer "B.Cu") (net 2))
+  (segment (start 76.8135 65.067) (end 76.8135 60.198) (width 0.25) (layer "B.Cu") (net 2))
+  (segment (start 74.821 54.033) (end 74.821 57.420604) (width 0.25) (layer "B.Cu") (net 2))
+  (segment (start 73.025 65.2995) (end 73.025 64.029) (width 0.25) (layer "B.Cu") (net 2))
+  (segment (start 71.247 67.0775) (end 73.025 65.2995) (width 0.25) (layer "B.Cu") (net 2))
+  (segment (start 74.46625 62.57025) (end 74.76625 62.57025) (width 0.25) (layer "B.Cu") (net 3))
+  (segment (start 74.46625 64.66575) (end 74.46625 62.57025) (width 0.25) (layer "B.Cu") (net 3))
+  (segment (start 75.84125 59.07725) (end 74.021 57.257) (width 0.25) (layer "B.Cu") (net 3))
+  (segment (start 75.84125 61.49525) (end 75.84125 59.07725) (width 0.25) (layer "B.Cu") (net 3))
+  (segment (start 74.803 65.0025) (end 74.46625 64.66575) (width 0.25) (layer "B.Cu") (net 3))
+  (segment (start 74.021 57.257) (end 74.021 54.033) (width 0.25) (layer "B.Cu") (net 3))
+  (segment (start 74.76625 62.57025) (end 75.84125 61.49525) (width 0.25) (layer "B.Cu") (net 3))
+  (segment (start 78.486 60.198) (end 78.8885 60.198) (width 0.25) (layer "B.Cu") (net 4))
+  (segment (start 75.621 54.033) (end 75.621 57.333) (width 0.25) (layer "B.Cu") (net 4))
+  (segment (start 75.621 57.333) (end 78.486 60.198) (width 0.25) (layer "B.Cu") (net 4))
+  (segment (start 78.8885 60.198) (end 78.8885 60.0925) (width 0.25) (layer "B.Cu") (net 4))
   (segment (start 46.1 69.05625) (end 58.549 69.05625) (width 0.25) (layer "B.Cu") (net 6))
   (segment (start 42.74375 59.76175) (end 42.799 59.817) (width 0.25) (layer "F.Cu") (net 7))

Commit message: Added ground plane
Parts:
- moved C1 1.48 mm to (70.5, 64.8)
- moved C2 1.48 mm to (74.0, 64.8)
- moved C6 1.48 mm to (77.1, 58.9)
- moved Y1 1.48 mm to (72.3, 60.2)
Routing:
- net +5V: track 7.86 -> 6.02 mm
- net /XTAL1: track 13.4 -> 11.8 mm
- net /XTAL2: track 12.6 -> 11.0 mm
- net GND: track 26.9 -> 25.4 mm, vias 0 -> 3
- added copper zone on B.Cu, net GND
- added copper zone on F.Cu, net GND
Changed lines of the file:
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@@
   )
   (footprint "Crystal:Crystal_SMD_3225-4Pin_3.2x2.5mm_HandSoldering" (layer "B.Cu")
-    (at 73.01625 61.42025)
+    (at 72.25425 60.15025)
     (descr "SMD Crystal SERIES SMD3225/4 http://www.txccrystal.com/images/pdf/7m-accuracy.pdf, hand-soldering, 3.2x2.5mm^2 package")
     (tags "SMD SMT crystal hand-soldering")
@@
   )
   (footprint "Capacitor_SMD:C_0805_2012Metric_Pad1.18x1.45mm_HandSolder" (layer "B.Cu")
-    (at 71.247 66.04 -90)
+    (at 70.485 64.77 -90)
     (descr "Capacitor SMD 0805 (2012 Metric), square (rectangular) end terminal, IPC_7351 nominal with elongated pad for handsoldering. (Body size source: IPC-SM-782 page 76, https://www.pcb-3d.com/wordpress/wp-content/uploads/ipc-sm-782a_amendment_1_and_2.pdf, https://docs.google.com/spreadsheets/d/1BsfQQcO9C6DZCsRaXUlFlo91Tg2WpOkGARC1WS5S8t0/edit?usp=sharing), generated with kicad-footprint-generator")
     (tags "capacitor handsolder")
@@
   )
   (footprint "Capacitor_SMD:C_0805_2012Metric_Pad1.18x1.45mm_HandSolder" (layer "B.Cu")
-    (at 74.803 66.04 -90)
+    (at 74.041 64.77 -90)
     (descr "Capacitor SMD 0805 (2012 Metric), square (rectangular) end terminal, IPC_7351 nominal with elongated pad for handsoldering. (Body size source: IPC-SM-782 page 76, https://www.pcb-3d.com/wordpress/wp-content/uploads/ipc-sm-782a_amendment_1_and_2.pdf, https://docs.google.com/spreadsheets/d/1BsfQQcO9C6DZCsRaXUlFlo91Tg2WpOkGARC1WS5S8t0/edit?usp=sharing), generated with kicad-footprint-generator")
     (tags "capacitor handsolder")
@@
   )
   (footprint "Capacitor_SMD:C_0805_2012Metric_Pad1.18x1.45mm_HandSolder" (layer "B.Cu")
-    (at 77.851 60.198 180)
+    (at 77.089 58.928 180)
     (descr "Capacitor SMD 0805 (2012 Metric), square (rectangular) end terminal, IPC_7351 nominal with elongated pad for handsoldering. (Body size source: IPC-SM-782 page 76, https://www.pcb-3d.com/wordpress/wp-content/uploads/ipc-sm-782a_amendment_1_and_2.pdf, https://docs.google.com/spreadsheets/d/1BsfQQcO9C6DZCsRaXUlFlo91Tg2WpOkGARC1WS5S8t0/edit?usp=sharing), generated with kicad-footprint-generator")
     (tags "capacitor handsolder")
@@
   (gr_line (start 37.30625 149.225) (end 110.33125 149.225) (layer "Edge.Cuts") (width 0.1))
   (gr_line (start 114.3 53.18125) (end 112.7125 53.18125) (layer "Edge.Cuts") (width 0.1))
-  (segment (start 69.977 61.341) (end 71.04775 60.27025) (width 0.25) (layer "B.Cu") (net 1))
-  (segment (start 73.221 57.335) (end 73.221 54.033) (width 0.25) (layer "B.Cu") (net 1))
-  (segment (start 71.56625 58.98975) (end 73.221 57.335) (width 0.25) (layer "B.Cu") (net 1))
-  (segment (start 69.977 64.135) (end 69.977 61.341) (width 0.25) (layer "B.Cu") (net 1))
-  (segment (start 71.04775 60.27025) (end 71.56625 60.27025) (width 0.25) (layer "B.Cu") (net 1))
-  (segment (start 71.56625 58.98975) (end 71.56625 60.27025) (width 0.25) (layer "B.Cu") (net 1))
-  (segment (start 70.8445 65.0025) (end 69.977 64.135) (width 0.25) (layer "B.Cu") (net 1))
-  (segment (start 71.247 65.0025) (end 70.8445 65.0025) (width 0.25) (layer "B.Cu") (net 1))
-  (segment (start 74.821 57.420604) (end 75.248198 57.847802) (width 0.25) (layer "B.Cu") (net 2))
-  (segment (start 74.803 67.0775) (end 76.8135 65.067) (width 0.25) (layer "B.Cu") (net 2))
-  (segment (start 76.8135 59.413104) (end 75.248198 57.847802) (width 0.25) (layer "B.Cu") (net 2))
-  (segment (start 76.8135 60.198) (end 76.8135 59.413104) (width 0.25) (layer "B.Cu") (net 2))
-  (segment (start 74.31625 60.27025) (end 72.01625 62.57025) (width 0.25) (layer "B.Cu") (net 2))
-  (segment (start 73.025 64.029) (end 71.56625 62.57025) (width 0.25) (layer "B.Cu") (net 2))
-  (segment (start 72.01625 62.57025) (end 71.56625 62.57025) (width 0.25) (layer "B.Cu") (net 2))
-  (segment (start 74.46625 60.27025) (end 74.31625 60.27025) (width 0.25) (layer "B.Cu") (net 2))
-  (segment (start 73.025 65.2995) (end 74.803 67.0775) (width 0.25) (layer "B.Cu") (net 2))
-  (segment (start 76.8135 65.067) (end 76.8135 60.198) (width 0.25) (layer "B.Cu") (net 2))
-  (segment (start 74.821 54.033) (end 74.821 57.420604) (width 0.25) (layer "B.Cu") (net 2))
-  (segment (start 73.025 65.2995) (end 73.025 64.029) (width 0.25) (layer "B.Cu") (net 2))
-  (segment (start 71.247 67.0775) (end 73.025 65.2995) (width 0.25) (layer "B.Cu") (net 2))
-  (segment (start 74.46625 62.57025) (end 74.76625 62.57025) (width 0.25) (layer "B.Cu") (net 3))
-  (segment (start 74.46625 64.66575) (end 74.46625 62.57025) (width 0.25) (layer "B.Cu") (net 3))
-  (segment (start 75.84125 59.07725) (end 74.021 57.257) (width 0.25) (layer "B.Cu") (net 3))
-  (segment (start 75.84125 61.49525) (end 75.84125 59.07725) (width 0.25) (layer "B.Cu") (net 3))
-  (segment (start 74.803 65.0025) (end 74.46625 64.66575) (width 0.25) (layer "B.Cu") (net 3))
-  (segment (start 74.021 57.257) (end 74.021 54.033) (width 0.25) (layer "B.Cu") (net 3))
-  (segment (start 74.76625 62.57025) (end 75.84125 61.49525) (width 0.25) (layer "B.Cu") (net 3))
-  (segment (start 78.486 60.198) (end 78.8885 60.198) (width 0.25) (layer "B.Cu") (net 4))
-  (segment (start 75.621 54.033) (end 75.621 57.333) (width 0.25) (layer "B.Cu") (net 4))
-  (segment (start 75.621 57.333) (end 78.486 60.198) (width 0.25) (layer "B.Cu") (net 4))
-  (segment (start 78.8885 60.198) (end 78.8885 60.0925) (width 0.25) (layer "B.Cu") (net 4))
+  (segment (start 70.66675 59.00025) (end 70.80425 59.00025) (width 0.25) (layer "B.Cu") (net 1))
+  (segment (start 70.485 63.7325) (end 69.42925 62.67675) (width 0.25) (layer "B.Cu") (net 1))
+  (segment (start 70.80425 59.00025) (end 73.221 56.5835) (width 0.25) (layer "B.Cu") (net 1))
+  (segment (start 73.221 56.5835) (end 73.221 54.033) (width 0.25) (layer "B.Cu") (net 1))
+  (segment (start 69.42925 60.23775) (end 70.66675 59.00025) (width 0.25) (layer "B.Cu") (net 1))
+  (segment (start 69.42925 62.67675) (end 69.42925 60.23775) (width 0.25) (layer "B.Cu") (net 1))
+  (via (at 70.485 67.437) (size 0.8) (drill 0.4) (layers "F.Cu" "B.Cu") (free) (net 2))
+  (via (at 74.041 67.437) (size 0.8) (drill 0.4) (layers "F.Cu" "B.Cu") (free) (net 2))
+  (via (at 73.66 57.277) (size 0.8) (drill 0.4) (layers "F.Cu" "B.Cu") (free) (net 2))
+  (segment (start 70.7175 65.8075) (end 72.39 64.135) (width 0.25) (layer "B.Cu") (net 2))
+  (segment (start 72.39 62.886) (end 70.80425 61.30025) (width 0.25) (layer "B.Cu") (net 2))
+  (segment (start 73.40425 59.00025) (end 71.10425 61.30025) (width 0.25) (layer "B.Cu") (net 2))
+  (segment (start 74.821 56.533) (end 74.821 54.033) (width 0.25) (layer "B.Cu") (net 2))
+  (segment (start 76.0515 57.7635) (end 74.821 56.533) (width 0.25) (layer "B.Cu") (net 2))
+  (segment (start 73.70425 59.00025) (end 73.40425 59.00025) (width 0.25) (layer "B.Cu") (net 2))
+  (segment (start 76.0515 58.928) (end 76.0515 57.7635) (width 0.25) (layer "B.Cu") (net 2))
+  (segment (start 70.485 65.8075) (end 70.7175 65.8075) (width 0.25) (layer "B.Cu") (net 2))
+  (segment (start 76.0515 63.347673) (end 76.0515 58.928) (width 0.25) (layer "B.Cu") (net 2))
+  (segment (start 71.10425 61.30025) (end 70.80425 61.30025) (width 0.25) (layer "B.Cu") (net 2))
+  (segment (start 74.041 65.8075) (end 74.041 65.358173) (width 0.25) (layer "B.Cu") (net 2))
+  (segment (start 72.39 64.135) (end 72.39 62.886) (width 0.25) (layer "B.Cu") (net 2))
+  (segment (start 74.041 65.786) (end 72.39 64.135) (width 0.25) (layer "B.Cu") (net 2))
+  (segment (start 74.041 65.8075) (end 74.041 65.786) (width 0.25) (layer "B.Cu") (net 2))
+  (segment (start 74.041 65.358173) (end 76.0515 63.347673) (width 0.25) (layer "B.Cu") (net 2))
+  (segment (start 74.041 63.7325) (end 73.70425 63.39575) (width 0.25) (layer "B.Cu") (net 3))
+  (segment (start 74.00425 61.30025) (end 73.70425 61.30025) (width 0.25) (layer "B.Cu") (net 3))
+  (segment (start 73.70425 63.39575) (end 73.70425 61.30025) (width 0.25) (layer "B.Cu") (net 3))
+  (segment (start 74.021 54.033) (end 74.021 56.495) (width 0.25) (layer "B.Cu") (net 3))
+  (segment (start 75.07925 60.22525) (end 74.00425 61.30025) (width 0.25) (layer "B.Cu") (net 3))
+  (segment (start 75.07925 57.55325) (end 75.07925 60.22525) (width 0.25) (layer "B.Cu") (net 3))
+  (segment (start 74.021 56.495) (end 75.07925 57.55325) (width 0.25) (layer "B.Cu") (net 3))
+  (segment (start 75.621 56.571) (end 75.621 54.033) (width 0.25) (layer "B.Cu") (net 4))
+  (segment (start 77.978 58.928) (end 75.621 56.571) (width 0.25) (layer "B.Cu") (net 4))
+  (segment (start 78.1265 58.928) (end 77.978 58.928) (width 0.25) (layer "B.Cu") (net 4))
   (segment (start 46.1 69.05625) (end 58.549 69.05625) (width 0.25) (layer "B.Cu") (net 6))
   (segment (start 42.74375 59.76175) (end 42.799 59.817) (width 0.25) (layer "F.Cu") (net 7))
@@
   (segment (start 97.584999 47.228) (end 96.809999 46.453) (width 0.2) (layer "B.Cu") (net 61))
   (segment (start 106.00125 47.58125) (end 104.97625 46.55625) (width 0.2) (layer "B.Cu") (net 61))
+  (zone (net 2) (net_name "GND") (layer "F.Cu") (hatch edge 0.508)
+    (connect_pads (clearance 0.508))
+    (min_thickness 0.254) (filled_areas_thickness no)
+    (fill yes (thermal_gap 0.508) (thermal_bridge_width 0.508))
+    (polygon
+      (pts
+        (xy 79.249259 68.20968)
+        (xy 68.324454 68.20692)
+        (xy 68.197744 55.375568)
+        (xy 72.770185 55.371952)
+        (xy 72.898 53.213)
+        (xy 74.421123 53.213573)
+        (xy 74.547309 55.372621)
+        (xy 79.122549 55.379679)
+      )
+    )
+  )
+  (zone (net 2) (net_name "GND") (layer "B.Cu") (hatch edge 0.508)
+    (connect_pads (clearance 0.508))
+    (min_thickness 0.254) (filled_areas_thickness no)
+    (fill yes (thermal_gap 0.508) (thermal_bridge_width 0.508))
+    (polygon
+      (pts
+        (xy 79.250516 68.20176)
+        (xy 68.325711 68.199)
+        (xy 68.199 55.372)
+        (xy 79.123805 55.376111)
+      )
+    )
+  )
 )
