File: keypad/keypad.kicad_pcb (KiCad board)
At the start: 2 copper layers, 78.6 x 111.1 mm, 59 parts, among them J1 AVR-ISP-6, SW1 num, SW10 #5, SW11 #6, SW12 plu1, SW13 #1, SW14 #2, SW15 #3, SW16 ent0, SW17 #0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

Commit message: Routed USB VCC
Routing:
- net GND: track 25.4 -> 58.6 mm
- net VCC: track 0.00 -> 20.1 mm, vias 0 -> 2
- net Net-(R6-Pad2): track 0.00 -> 6.00 mm
- net Net-(R5-Pad2): track 0.00 -> 5.82 mm
Changed lines of the file:
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@@
   (via (at 73.66 57.277) (size 0.8) (drill 0.4) (layers "F.Cu" "B.Cu") (free) (net 2))
   (segment (start 70.7175 65.8075) (end 72.39 64.135) (width 0.25) (layer "B.Cu") (net 2))
+  (segment (start 103.96875 50.05625) (end 102.225 51.8) (width 0.25) (layer "B.Cu") (net 2))
+  (segment (start 107.835 43.60625) (end 108.93 42.51125) (width 0.25) (layer "B.Cu") (net 2))
   (segment (start 72.39 62.886) (end 70.80425 61.30025) (width 0.25) (layer "B.Cu") (net 2))
+  (segment (start 107.515 43.60625) (end 107.835 43.60625) (width 0.25) (layer "B.Cu") (net 2))
+  (segment (start 107.515 50.05625) (end 103.96875 50.05625) (width 0.25) (layer "B.Cu") (net 2))
   (segment (start 73.40425 59.00025) (end 71.10425 61.30025) (width 0.25) (layer "B.Cu") (net 2))
+  (segment (start 113.11 42.51125) (end 108.93 42.51125) (width 0.25) (layer "B.Cu") (net 2))
   (segment (start 74.821 56.533) (end 74.821 54.033) (width 0.25) (layer "B.Cu") (net 2))
   (segment (start 76.0515 57.7635) (end 74.821 56.533) (width 0.25) (layer "B.Cu") (net 2))
   (segment (start 73.70425 59.00025) (end 73.40425 59.00025) (width 0.25) (layer "B.Cu") (net 2))
+  (segment (start 107.835 50.05625) (end 108.93 51.15125) (width 0.25) (layer "B.Cu") (net 2))
+  (segment (start 103.3305 41.8625) (end 102.225 41.8625) (width 0.25) (layer "B.Cu") (net 2))
   (segment (start 76.0515 58.928) (end 76.0515 57.7635) (width 0.25) (layer "B.Cu") (net 2))
+  (segment (start 105.07425 43.60625) (end 103.3305 41.8625) (width 0.25) (layer "B.Cu") (net 2))
   (segment (start 70.485 65.8075) (end 70.7175 65.8075) (width 0.25) (layer "B.Cu") (net 2))
   (segment (start 76.0515 63.347673) (end 76.0515 58.928) (width 0.25) (layer "B.Cu") (net 2))
   (segment (start 71.10425 61.30025) (end 70.80425 61.30025) (width 0.25) (layer "B.Cu") (net 2))
+  (segment (start 98.66875 50.52625) (end 99.81 49.385) (width 0.25) (layer "B.Cu") (net 2))
+  (segment (start 107.515 43.60625) (end 105.07425 43.60625) (width 0.25) (layer "B.Cu") (net 2))
   (segment (start 74.041 65.8075) (end 74.041 65.358173) (width 0.25) (layer "B.Cu") (net 2))
+  (segment (start 108.93 51.15125) (end 113.11 51.15125) (width 0.25) (layer "B.Cu") (net 2))
+  (segment (start 98.66875 52.3875) (end 98.66875 50.52625) (width 0.25) (layer "B.Cu") (net 2))
   (segment (start 72.39 64.135) (end 72.39 62.886) (width 0.25) (layer "B.Cu") (net 2))
   (segment (start 74.041 65.786) (end 72.39 64.135) (width 0.25) (layer "B.Cu") (net 2))
+  (segment (start 102.225 51.8) (end 99.81 49.385) (width 0.25) (layer "B.Cu") (net 2))
+  (segment (start 107.515 50.05625) (end 107.835 50.05625) (width 0.25) (layer "B.Cu") (net 2))
   (segment (start 74.041 65.8075) (end 74.041 65.786) (width 0.25) (layer "B.Cu") (net 2))
   (segment (start 74.041 65.358173) (end 76.0515 63.347673) (width 0.25) (layer "B.Cu") (net 2))
+  (segment (start 99.81 49.385) (end 99.81 47.228) (width 0.25) (layer "B.Cu") (net 2))
   (segment (start 74.041 63.7325) (end 73.70425 63.39575) (width 0.25) (layer "B.Cu") (net 3))
   (segment (start 74.00425 61.30025) (end 73.70425 61.30025) (width 0.25) (layer "B.Cu") (net 3))
@@
   (segment (start 99.89375 135.7) (end 99.89375 145.075) (width 0.25) (layer "B.Cu") (net 29))
   (segment (start 99.89375 145.075) (end 100.075 145.25625) (width 0.25) (layer "B.Cu") (net 29))
+  (segment (start 104.356923 49.249423) (end 104.38875 49.28125) (width 0.25) (layer "F.Cu") (net 30))
+  (segment (start 104.356923 44.38125) (end 104.356923 49.249423) (width 0.25) (layer "F.Cu") (net 30))
+  (via (at 104.356923 44.38125) (size 0.8) (drill 0.4) (layers "F.Cu" "B.Cu") (net 30))
+  (via (at 104.38875 49.28125) (size 0.8) (drill 0.4) (layers "F.Cu" "B.Cu") (net 30))
+  (segment (start 99.625 41.275) (end 99.625 41.459) (width 0.25) (layer "B.Cu") (net 30))
+  (segment (start 99.625 41.459) (end 101.092 42.926) (width 0.25) (layer "B.Cu") (net 30))
+  (segment (start 106.17725 49.28125) (end 104.38875 49.28125) (width 0.25) (layer "B.Cu") (net 30))
+  (segment (start 101.092 42.926) (end 100.01 44.008) (width 0.25) (layer "B.Cu") (net 30))
+  (segment (start 107.515 49.28125) (end 106.17725 49.28125) (width 0.25) (layer "B.Cu") (net 30))
+  (segment (start 102.901673 42.926) (end 101.092 42.926) (width 0.25) (layer "B.Cu") (net 30))
+  (segment (start 107.515 44.38125) (end 104.356923 44.38125) (width 0.25) (layer "B.Cu") (net 30))
+  (segment (start 104.356923 44.38125) (end 102.901673 42.926) (width 0.25) (layer "B.Cu") (net 30))
+  (segment (start 100.01 44.008) (end 100.01 45.228) (width 0.25) (layer "B.Cu") (net 30))
+  (segment (start 104.374529 49.28125) (end 104.358711 49.265432) (width 0.25) (layer "B.Cu") (net 30))
+  (segment (start 104.38875 49.28125) (end 104.374529 49.28125) (width 0.25) (layer "B.Cu") (net 30))
   (segment (start 83.23525 45.908) (end 83.93125 45.212) (width 0.2) (layer "B.Cu") (net 35))
   (segment (start 80.246001 45.733) (end 80.421001 45.908) (width 0.2) (layer "B.Cu") (net 35))
@@
   (segment (start 80.246001 46.533) (end 80.421001 46.358) (width 0.2) (layer "B.Cu") (net 36))
   (segment (start 79.121 46.533) (end 80.246001 46.533) (width 0.2) (layer "B.Cu") (net 36))
+  (segment (start 107.49 48.55625) (end 103.46875 48.55625) (width 0.25) (layer "B.Cu") (net 38))
+  (segment (start 103.46875 48.55625) (end 102.225 49.8) (width 0.25) (layer "B.Cu") (net 38))
+  (segment (start 107.515 48.58125) (end 107.49 48.55625) (width 0.25) (layer "B.Cu") (net 38))
+  (segment (start 107.515 45.58125) (end 103.94375 45.58125) (width 0.25) (layer "B.Cu") (net 39))
+  (segment (start 103.94375 45.58125) (end 102.225 43.8625) (width 0.25) (layer "B.Cu") (net 39))
   (segment (start 47.74375 125.675) (end 57.26875 135.2) (width 0.25) (layer "F.Cu") (net 40))
   (segment (start 47.74375 116.15) (end 47.74375 125.675) (width 0.25) (layer "F.Cu") (net 40))
